File: hardware/frontpanel.brd (EAGLE design)
At the start: 100 x 80 mm, 72 parts, among them IC1 STM32F103VET, Q1 8MHz, SW1 EC12E_SW, X1 MINI-USB_SHIELD4P-85-32004-00X

Commit message: board update
Parts:
- removed 22: (no value), switch-omron:SMD
- removed D23: 1N4148, diode:SOD323-W
- removed IC3: (no value), v-reg-3:SOT223
- removed SV1: (no value), con-lsta:FE20-2
- added IC2: VREG-TS1117CW-3V3, we-power:SOT223
- added SV2: (no value), con-lsta:FE06
- added SV3: (no value), con-lsta:FE08
- R4: device resistor:R0603 -> resistor:R1206
Connections:
- removed net EXT0: IC1.15, SV1.9
- removed net EXT1: IC1.16, SV1.10
- removed net EXT10: IC1.30, SV1.19
- removed net EXT11: IC1.31, SV1.20
- removed net EXT12: IC1.32, SV1.21
- removed net EXT13: IC1.33, SV1.22
- removed net EXT14: IC1.34, SV1.23
- removed net EXT15: IC1.35, SV1.24
- removed net EXT16: IC1.36, SV1.25
- removed net EXT17: IC1.37, SV1.26
- removed net EXT18: IC1.38, SV1.27
- removed net EXT19: IC1.39, SV1.28
- removed net EXT2: IC1.17, SV1.11
- removed net EXT20: IC1.40, SV1.29
- removed net EXT21: IC1.41, SV1.30
- removed net EXT22: IC1.42, SV1.31
- removed net EXT23: IC1.43, SV1.32
- removed net EXT24: IC1.44, SV1.33
- removed net EXT25: IC1.45, SV1.34
- removed net EXT26: IC1.46, SV1.35
- removed net EXT27: IC1.47, SV1.36
- removed net EXT28: IC1.48, SV1.38
- removed net EXT3: IC1.18, SV1.12
- removed net EXT5: IC1.23, SV1.14
- removed net EXT6: IC1.24, SV1.15
- removed net EXT7: IC1.25, SV1.16
- removed net EXT8: IC1.26, SV1.17
- removed net EXT9: IC1.29, SV1.18
- removed net N$29: 22.4, D23.A
- removed net N$75: 18.1, 22.2
- removed net NEGATIV: H1.B4,3, SV1.1, SV1.2, SV1.3, SV1.4
- removed net POSITIV: H2.B4,3, SV1.5, SV1.6, SV1.7, SV1.8
- new net N$31: IC1.31, SV2.5
- new net N$32: IC1.30, SV2.4
- new net N$37: IC1.32, SV2.3
- new net OUT+: H2.B4,3, SV3.1, SV3.2, SV3.3, SV3.4
- new net OUT-: H1.B4,3, SV3.5, SV3.6, SV3.7, SV3.8
- net +3V3: now also IC2.2, IC2.4, SV2.2; no longer IC3.2, SV1.37
- net +5V: now also IC2.3, SV2.1; no longer IC3.3, SV1.39
- net EXT4: no longer SV1.13
- net GND: now also IC2.1, SV2.6; no longer IC3.1, SV1.40
- net SWITCH_OUT6: no longer D23.C
Routing:
- net POSITIV: track 147.5 -> 0.00 mm
- net NEGATIV: track 80.9 -> 0.00 mm
- net EXT1: track 38.3 -> 0.00 mm
- net EXT0: track 36.5 -> 0.00 mm
- net EXT3: track 35.9 -> 0.00 mm
- net EXT2: track 34.0 -> 0.00 mm
- net EXT5: track 30.0 -> 0.00 mm
- net N$32: track 0.00 -> 27.3 mm
- net EXT7: track 27.2 -> 0.00 mm
- net EXT9: track 25.8 -> 0.00 mm
- net EXT6: track 25.6 -> 0.00 mm
- net EXT11: track 25.1 -> 0.00 mm
- net EXT28: track 25.0 -> 0.00 mm
- net EXT13: track 24.5 -> 0.00 mm
- net EXT27: track 24.1 -> 0.00 mm
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- added copper zone on layer 1, net OUT+
- added copper zone on layer 16, net OUT+
- added copper zone on layer 1, net OUT-
- added copper zone on layer 16, net OUT-
Other:
- outline, holes or cut-outs redrawn

Commit message: PCB markings
Connections:
- net N$31 renamed MISO
- net N$32 renamed SCK
- net N$37 renamed MOSI
- net N$73 renamed TX
- net N$74 renamed RX
Other:
- board text added: "-> 5V"
- board text added: "3V3"
- board text added: "<- 3V3"
- board text added: "Battery simulator"
- board text added: "Frontpanel 04/2017"
- board text added: "GND"
- board text added: "MISO"
- board text added: "MOSI"
- board text added: "NRST"
- board text added: "OUT+"
- board text added: "OUT-"
- board text added: "RX"
- board text added: "SCK"
- board text added: "SWCLK"
- board text added: "SWDIO"
- board text added: "TX"
- board text added: "github.com/jankae/battery-sim"

Commit message: minor PCB changes
Parts:
- removed C16, C17: 100µ, rcl:E2,5-6
- added C10, C9: 100u, rcl:153CLV-0505
- moved IC2 40.1 mm to (55.2, 11.7), turned to 180 degrees
- moved C15 39.7 mm to (56.5, 17.5)
- moved C14 29.5 mm to (59.7, 17.5), turned to 180 degrees
Connections:
- net +3V3: now also C10.+; no longer C16.+
- net +5V: now also C9.+; no longer C17.+
- net GND: now also C10.-, C9.-; no longer C16.-, C17.-
- net SWITCH_OUT6: now also IC1.36; no longer IC1.51
Routing:
- net +3V3: track 191.2 -> 152.9 mm
- net GND: track 288.7 -> 292.6 mm, vias 6 -> 8
- net SWITCH_OUT6: track 36.2 -> 32.5 mm
- net +5V: track 79.9 -> 76.7 mm, vias 2 -> 3
- net MOSI: track 23.6 -> 26.0 mm
Other:
- outline, holes or cut-outs redrawn

Commit message: final PCB corrections
Parts:
- added C11: 100n, resistormod:C0603K
- added PA0, PA1, PA2, PA3, PA4, PC0, PC1, PC2, PC3: (no value), wirepad:SMD1,27-2,54
- added R1, R5: 10k, resistor:R0603
Connections:
- new net ADC_5V: C11.1, IC1.35, R1.1, R5.2
- new net N$1: IC1.15, PC0.1
- new net N$29: IC1.16, PC1.1
- new net N$30: IC1.17, PC2.1
- new net N$31: IC1.18, PC3.1
- new net N$32: IC1.23, PA0.1
- new net N$37: IC1.24, PA1.1
- new net N$41: IC1.25, PA2.1
- new net N$45: IC1.26, PA3.1
- new net N$65: IC1.29, PA4.1
- net +5V: now also R1.2
- net GND: now also C11.2, R5.1
Routing:
- net ADC_5V: track 0.00 -> 36.0 mm, vias 0 -> 4
- net N$31: track 0.00 -> 11.8 mm
- net N$30: track 0.00 -> 11.2 mm
- net N$29: track 0.00 -> 10.6 mm
- net N$32: track 0.00 -> 10.6 mm
- net N$1: track 0.00 -> 10.0 mm
- net N$37: track 0.00 -> 10.0 mm
- net N$41: track 0.00 -> 7.27 mm
- net N$45: track 0.00 -> 6.07 mm
- net N$65: track 0.00 -> 4.63 mm
- net +5V: track 76.7 -> 80.1 mm
- net GND: track 292.6 -> 294.7 mm, vias 8 -> 9
