File: hardware/frontpanel.sch (EAGLE design)
At the start: 72 parts, among them IC1 STM32F103VET, Q1 8MHz, SW1 EC12E_SW, X1 MINI-USB_SHIELD4P-85-32004-00X

Commit message: board update
Parts:
- removed 22: (no value), switch-omron:10-XXSMD
- removed D23: 1N4148, diode:DIODE-SOD323-W
- removed IC3: (no value), v-reg-3:LM1117
- removed SV1: (no value), con-lsta:FE20-2
- added IC2: VREG-TS1117CW-3V3, we-power:VREG-TS1117CW-3V3
- added SV2: (no value), con-lsta:FE06-1
- added SV3: (no value), con-lsta:FE08-1
- R4: device resistor:R-EU_R0603 -> resistor:R-EU_R1206
Connections:
- removed net EXT0: IC1MCU.PC0, SV1.9
- removed net EXT1: IC1MCU.PC1, SV1.10
- removed net EXT10: IC1MCU.PA5, SV1.19
- removed net EXT11: IC1MCU.PA6, SV1.20
- removed net EXT12: IC1MCU.PA7, SV1.21
- removed net EXT13: IC1MCU.PC4, SV1.22
- removed net EXT14: IC1MCU.PC5, SV1.23
- removed net EXT15: IC1MCU.PB0, SV1.24
- removed net EXT16: IC1MCU.PB1, SV1.25
- removed net EXT17: IC1MCU.PB2, SV1.26
- removed net EXT18: IC1MCU.PE7, SV1.27
- removed net EXT19: IC1MCU.PE8, SV1.28
- removed net EXT2: IC1MCU.PC2, SV1.11
- removed net EXT20: IC1MCU.PE9, SV1.29
- removed net EXT21: IC1MCU.PE10, SV1.30
- removed net EXT22: IC1MCU.PE11, SV1.31
- removed net EXT23: IC1MCU.PE12, SV1.32
- removed net EXT24: IC1MCU.PE13, SV1.33
- removed net EXT25: IC1MCU.PE14, SV1.34
- removed net EXT26: IC1MCU.PE15, SV1.35
- removed net EXT27: IC1MCU.PB10, SV1.36
- removed net EXT28: IC1MCU.PB11, SV1.38
- removed net EXT3: IC1MCU.PC3, SV1.12
- removed net EXT5: IC1MCU.PA0-WKUP, SV1.14
- removed net EXT6: IC1MCU.PA1, SV1.15
- removed net EXT7: IC1MCU.PA2, SV1.16
- removed net EXT8: IC1MCU.PA3, SV1.17
- removed net EXT9: IC1MCU.PA4, SV1.18
- removed net N$29: 22.P1, D23.A
- removed net N$75: 18.S, 22.S1
- removed net NEGATIV: H1.MOUNT, SV1.1, SV1.2, SV1.3, SV1.4
- removed net POSITIV: H2.MOUNT, SV1.5, SV1.6, SV1.7, SV1.8
- new net N$31: IC1MCU.PA6, SV2.5
- new net N$32: IC1MCU.PA5, SV2.4
- new net N$37: IC1MCU.PA7, SV2.3
- new net OUT+: H2.MOUNT, SV3.1, SV3.2, SV3.3, SV3.4
- new net OUT-: H1.MOUNT, SV3.5, SV3.6, SV3.7, SV3.8
- net +3V3: now also IC2.VOUT, SV2.2; no longer IC3.OUT, SV1.37
- net +5V: now also IC2.VIN, SV2.1; no longer IC3.IN, SV1.39
- net EXT4: no longer SV1.13
- net GND: now also IC2.GND, SV2.6; no longer IC3.GND, SV1.40
- net SWITCH_OUT6: no longer D23.C
Other:
- moved on the sheet: C14, C17, H1, H2

Commit message: PCB markings
Connections:
- net N$31 renamed MISO
- net N$32 renamed SCK
- net N$37 renamed MOSI
- net N$73 renamed TX
- net N$74 renamed RX
Changed lines of the file:
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@@
 <grid distance="0.1" unitdist="inch" unit="inch" style="lines" multiple="1" display="no" altdistance="0.01" altunitdist="inch" altunit="inch"/>
 <layers>
-<layer number="1" name="Top" color="4" fill="1" visible="yes" active="no"/>
-<layer number="2" name="Route2" color="1" fill="3" visible="yes" active="no"/>
-<layer number="3" name="Route3" color="4" fill="3" visible="yes" active="no"/>
-<layer number="14" name="Route14" color="1" fill="6" visible="yes" active="no"/>
-<layer number="15" name="Route15" color="4" fill="6" visible="yes" active="no"/>
-<layer number="16" name="Bottom" color="1" fill="1" visible="yes" active="no"/>
-<layer number="17" name="Pads" color="2" fill="1" visible="yes" active="no"/>
-<layer number="18" name="Vias" color="2" fill="1" visible="yes" active="no"/>
-<layer number="19" name="Unrouted" color="6" fill="1" visible="yes" active="no"/>
-<layer number="20" name="Dimension" color="15" fill="1" visible="yes" active="no"/>
-<layer number="21" name="tPlace" color="7" fill="1" visible="yes" active="no"/>
-<layer number="22" name="bPlace" color="7" fill="1" visible="yes" active="no"/>
-<layer number="23" name="tOrigins" color="15" fill="1" visible="yes" active="no"/>
-<layer number="24" name="bOrigins" color="15" fill="1" visible="yes" active="no"/>
-<layer number="25" name="tNames" color="7" fill="1" visible="yes" active="no"/>
-<layer number="26" name="bNames" color="7" fill="1" visible="yes" active="no"/>
-<layer number="27" name="tValues" color="7" fill="1" visible="yes" active="no"/>
-<layer number="28" name="bValues" color="7" fill="1" visible="yes" active="no"/>
+<layer number="1" name="Top" color="4" fill="1" visible="no" active="no"/>
+<layer number="2" name="Route2" color="1" fill="3" visible="no" active="no"/>
+<layer number="3" name="Route3" color="4" fill="3" visible="no" active="no"/>
+<layer number="14" name="Route14" color="1" fill="6" visible="no" active="no"/>
+<layer number="15" name="Route15" color="4" fill="6" visible="no" active="no"/>
+<layer number="16" name="Bottom" color="1" fill="1" visible="no" active="no"/>
+<layer number="17" name="Pads" color="2" fill="1" visible="no" active="no"/>
+<layer number="18" name="Vias" color="2" fill="1" visible="no" active="no"/>
+<layer number="19" name="Unrouted" color="6" fill="1" visible="no" active="no"/>
+<layer number="20" name="Dimension" color="15" fill="1" visible="no" active="no"/>
+<layer number="21" name="tPlace" color="7" fill="1" visible="no" active="no"/>
+<layer number="22" name="bPlace" color="7" fill="1" visible="no" active="no"/>
+<layer number="23" name="tOrigins" color="15" fill="1" visible="no" active="no"/>
+<layer number="24" name="bOrigins" color="15" fill="1" visible="no" active="no"/>
+<layer number="25" name="tNames" color="7" fill="1" visible="no" active="no"/>
+<layer number="26" name="bNames" color="7" fill="1" visible="no" active="no"/>
+<layer number="27" name="tValues" color="7" fill="1" visible="no" active="no"/>
+<layer number="28" name="bValues" color="7" fill="1" visible="no" active="no"/>
 <layer number="29" name="tStop" color="7" fill="3" visible="no" active="no"/>
 <layer number="30" name="bStop" color="7" fill="6" visible="no" active="no"/>
@@
 <layer number="35" name="tGlue" color="7" fill="4" visible="no" active="no"/>
 <layer number="36" name="bGlue" color="7" fill="5" visible="no" active="no"/>
-<layer number="37" name="tTest" color="7" fill="1" visible="yes" active="no"/>
-<layer number="38" name="bTest" color="7" fill="1" visible="yes" active="no"/>
+<layer number="37" name="tTest" color="7" fill="1" visible="no" active="no"/>
+<layer number="38" name="bTest" color="7" fill="1" visible="no" active="no"/>
 <layer number="39" name="tKeepout" color="4" fill="11" visible="no" active="no"/>
 <layer number="40" name="bKeepout" color="1" fill="11" visible="no" active="no"/>
@@
 <layer number="44" name="Drills" color="7" fill="1" visible="no" active="no"/>
 <layer number="45" name="Holes" color="7" fill="1" visible="no" active="no"/>
-<layer number="46" name="Milling" color="3" fill="1" visible="yes" active="no"/>
-<layer number="47" name="Measures" color="7" fill="1" visible="yes" active="no"/>
-<layer number="48" name="Document" color="7" fill="1" visible="yes" active="no"/>
-<layer number="49" name="Reference" color="7" fill="1" visible="yes" active="no"/>
-<layer number="50" name="dxf" color="7" fill="1" visible="yes" active="no"/>
-<layer number="51" name="tDocu" color="7" fill="1" visible="yes" active="no"/>
-<layer number="52" name="bDocu" color="7" fill="1" visible="yes" active="no"/>
-<layer number="53" name="tGND_GNDA" color="7" fill="9" visible="yes" active="no"/>
-<layer number="54" name="bGND_GNDA" color="1" fill="9" visible="yes" active="no"/>
-<layer number="56" name="wert" color="7" fill="1" visible="yes" active="no"/>
+<layer number="46" name="Milling" color="3" fill="1" visible="no" active="no"/>
+<layer number="47" name="Measures" color="7" fill="1" visible="no" active="no"/>
+<layer number="48" name="Document" color="7" fill="1" visible="no" active="no"/>
+<layer number="49" name="Reference" color="7" fill="1" visible="no" active="no"/>
+<layer number="50" name="dxf" color="7" fill="1" visible="no" active="no"/>
+<layer number="51" name="tDocu" color="7" fill="1" visible="no" active="no"/>
+<layer number="52" name="bDocu" color="7" fill="1" visible="no" active="no"/>
+<layer number="53" name="tGND_GNDA" color="7" fill="9" visible="no" active="no"/>
+<layer number="54" name="bGND_GNDA" color="1" fill="9" visible="no" active="no"/>
+<layer number="56" name="wert" color="7" fill="1" visible="no" active="no"/>
 <layer number="90" name="Modules" color="5" fill="1" visible="yes" active="yes"/>
 <layer number="91" name="Nets" color="2" fill="1" visible="yes" active="yes"/>
@@
 </segment>
 </net>
-<net name="N$73" class="0">
+<net name="TX" class="0">
 <segment>
 <pinref part="UART" gate="A" pin="3"/>
@@
 </segment>
 </net>
-<net name="N$74" class="0">
+<net name="RX" class="0">
 <segment>
 <pinref part="UART" gate="A" pin="1"/>
@@
 </segment>
 </net>
-<net name="N$31" class="0">
+<net name="MISO" class="0">
 <segment>
 <pinref part="SV2" gate="G$1" pin="5"/>
@@
 </segment>
 </net>
-<net name="N$32" class="0">
+<net name="SCK" class="0">
 <segment>
 <pinref part="SV2" gate="G$1" pin="4"/>
@@
 </segment>
 </net>
-<net name="N$37" class="0">
+<net name="MOSI" class="0">
 <segment>
 <pinref part="SV2" gate="G$1" pin="3"/>

Commit message: minor PCB changes
Parts:
- removed C16, C17: 100µ, rcl:CPOL-EUE2.5-6
- added C10, C9: 100u, rcl:CPOL-EU153CLV-0505
Connections:
- net +3V3: now also C10.+; no longer C16.+
- net +5V: now also C9.+; no longer C17.+
- net GND: now also C10.-, C9.-; no longer C16.-, C17.-
- net SWITCH_OUT6: now also IC1MCU.PB1; no longer IC1MCU.PB12
Changed lines of the file:
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@@
 <grid distance="0.1" unitdist="inch" unit="inch" style="lines" multiple="1" display="no" altdistance="0.01" altunitdist="inch" altunit="inch"/>
 <layers>
-<layer number="1" name="Top" color="4" fill="1" visible="no" active="no"/>
-<layer number="2" name="Route2" color="1" fill="3" visible="no" active="no"/>
-<layer number="3" name="Route3" color="4" fill="3" visible="no" active="no"/>
-<layer number="14" name="Route14" color="1" fill="6" visible="no" active="no"/>
-<layer number="15" name="Route15" color="4" fill="6" visible="no" active="no"/>
-<layer number="16" name="Bottom" color="1" fill="1" visible="no" active="no"/>
-<layer number="17" name="Pads" color="2" fill="1" visible="no" active="no"/>
-<layer number="18" name="Vias" color="2" fill="1" visible="no" active="no"/>
-<layer number="19" name="Unrouted" color="6" fill="1" visible="no" active="no"/>
-<layer number="20" name="Dimension" color="15" fill="1" visible="no" active="no"/>
-<layer number="21" name="tPlace" color="7" fill="1" visible="no" active="no"/>
-<layer number="22" name="bPlace" color="7" fill="1" visible="no" active="no"/>
-<layer number="23" name="tOrigins" color="15" fill="1" visible="no" active="no"/>
-<layer number="24" name="bOrigins" color="15" fill="1" visible="no" active="no"/>
-<layer number="25" name="tNames" color="7" fill="1" visible="no" active="no"/>
-<layer number="26" name="bNames" color="7" fill="1" visible="no" active="no"/>
-<layer number="27" name="tValues" color="7" fill="1" visible="no" active="no"/>
-<layer number="28" name="bValues" color="7" fill="1" visible="no" active="no"/>
+<layer number="1" name="Top" color="4" fill="1" visible="yes" active="no"/>
+<layer number="2" name="Route2" color="1" fill="3" visible="yes" active="no"/>
+<layer number="3" name="Route3" color="4" fill="3" visible="yes" active="no"/>
+<layer number="14" name="Route14" color="1" fill="6" visible="yes" active="no"/>
+<layer number="15" name="Route15" color="4" fill="6" visible="yes" active="no"/>
+<layer number="16" name="Bottom" color="1" fill="1" visible="yes" active="no"/>
+<layer number="17" name="Pads" color="2" fill="1" visible="yes" active="no"/>
+<layer number="18" name="Vias" color="2" fill="1" visible="yes" active="no"/>
+<layer number="19" name="Unrouted" color="6" fill="1" visible="yes" active="no"/>
+<layer number="20" name="Dimension" color="15" fill="1" visible="yes" active="no"/>
+<layer number="21" name="tPlace" color="7" fill="1" visible="yes" active="no"/>
+<layer number="22" name="bPlace" color="7" fill="1" visible="yes" active="no"/>
+<layer number="23" name="tOrigins" color="15" fill="1" visible="yes" active="no"/>
+<layer number="24" name="bOrigins" color="15" fill="1" visible="yes" active="no"/>
+<layer number="25" name="tNames" color="7" fill="1" visible="yes" active="no"/>
+<layer number="26" name="bNames" color="7" fill="1" visible="yes" active="no"/>
+<layer number="27" name="tValues" color="7" fill="1" visible="yes" active="no"/>
+<layer number="28" name="bValues" color="7" fill="1" visible="yes" active="no"/>
 <layer number="29" name="tStop" color="7" fill="3" visible="no" active="no"/>
 <layer number="30" name="bStop" color="7" fill="6" visible="no" active="no"/>
@@
 <layer number="35" name="tGlue" color="7" fill="4" visible="no" active="no"/>
 <layer number="36" name="bGlue" color="7" fill="5" visible="no" active="no"/>
-<layer number="37" name="tTest" color="7" fill="1" visible="no" active="no"/>
-<layer number="38" name="bTest" color="7" fill="1" visible="no" active="no"/>
+<layer number="37" name="tTest" color="7" fill="1" visible="yes" active="no"/>
+<layer number="38" name="bTest" color="7" fill="1" visible="yes" active="no"/>
 <layer number="39" name="tKeepout" color="4" fill="11" visible="no" active="no"/>
 <layer number="40" name="bKeepout" color="1" fill="11" visible="no" active="no"/>
@@
 <layer number="44" name="Drills" color="7" fill="1" visible="no" active="no"/>
 <layer number="45" name="Holes" color="7" fill="1" visible="no" active="no"/>
-<layer number="46" name="Milling" color="3" fill="1" visible="no" active="no"/>
-<layer number="47" name="Measures" color="7" fill="1" visible="no" active="no"/>
-<layer number="48" name="Document" color="7" fill="1" visible="no" active="no"/>
-<layer number="49" name="Reference" color="7" fill="1" visible="no" active="no"/>
-<layer number="50" name="dxf" color="7" fill="1" visible="no" active="no"/>
-<layer number="51" name="tDocu" color="7" fill="1" visible="no" active="no"/>
-<layer number="52" name="bDocu" color="7" fill="1" visible="no" active="no"/>
-<layer number="53" name="tGND_GNDA" color="7" fill="9" visible="no" active="no"/>
-<layer number="54" name="bGND_GNDA" color="1" fill="9" visible="no" active="no"/>
-<layer number="56" name="wert" color="7" fill="1" visible="no" active="no"/>
+<layer number="46" name="Milling" color="3" fill="1" visible="yes" active="no"/>
+<layer number="47" name="Measures" color="7" fill="1" visible="yes" active="no"/>
+<layer number="48" name="Document" color="7" fill="1" visible="yes" active="no"/>
+<layer number="49" name="Reference" color="7" fill="1" visible="yes" active="no"/>
+<layer number="50" name="dxf" color="7" fill="1" visible="yes" active="no"/>
+<layer number="51" name="tDocu" color="7" fill="1" visible="yes" active="no"/>
+<layer number="52" name="bDocu" color="7" fill="1" visible="yes" active="no"/>
+<layer number="53" name="tGND_GNDA" color="7" fill="9" visible="yes" active="no"/>
+<layer number="54" name="bGND_GNDA" color="1" fill="9" visible="yes" active="no"/>
+<layer number="56" name="wert" color="7" fill="1" visible="yes" active="no"/>
 <layer number="90" name="Modules" color="5" fill="1" visible="yes" active="yes"/>
 <layer number="91" name="Nets" color="2" fill="1" visible="yes" active="yes"/>
@@
 <part name="C14" library="resistormod" deviceset="C-EU" device="C0603K" value="100n"/>
 <part name="C15" library="resistormod" deviceset="C-EU" device="C0603K" value="100n"/>
-<part name="C16" library="rcl" deviceset="CPOL-EU" device="E2.5-6" value="100µ"/>
-<part name="C17" library="rcl" deviceset="CPOL-EU" device="E2.5-6" value="100µ"/>
 <part name="13" library="switch-omron" deviceset="10-XX" device="SMD"/>
 <part name="14" library="switch-omron" deviceset="10-XX" device="SMD"/>
@@
 <part name="P+3" library="supply1" deviceset="+5V" device=""/>
 <part name="IC2" library="we-power" deviceset="VREG" device="-TS1117CW-3V3"/>
+<part name="C9" library="rcl" deviceset="CPOL-EU" device="153CLV-0505" value="100u"/>
+<part name="C10" library="rcl" deviceset="CPOL-EU" device="153CLV-0505" value="100u"/>
 </parts>
 <sheets>
@@
 <instance part="C14" gate="G$1" x="-22.86" y="167.64"/>
 <instance part="C15" gate="G$1" x="7.62" y="167.64"/>
-<instance part="C16" gate="G$1" x="17.78" y="167.64"/>
-<instance part="C17" gate="G$1" x="-33.02" y="167.64"/>
 <instance part="13" gate="1" x="-5.08" y="-88.9" rot="R270"/>
 <instance part="14" gate="1" x="17.78" y="-88.9" rot="R270"/>
@@
 <instance part="P+3" gate="1" x="200.66" y="60.96"/>
 <instance part="IC2" gate="IC" x="-7.62" y="172.72"/>
+<instance part="C9" gate="G$1" x="-33.02" y="167.64"/>
+<instance part="C10" gate="G$1" x="17.78" y="167.64"/>
 </instances>
 <busses>
@@
 <junction x="7.62" y="172.72"/>
 <wire x1="7.62" y1="172.72" x2="17.78" y2="172.72" width="0.1524" layer="91"/>
-<pinref part="C16" gate="G$1" pin="+"/>
 <wire x1="17.78" y1="172.72" x2="17.78" y2="170.18" width="0.1524" layer="91"/>
 <pinref part="+3V6" gate="G$1" pin="+3V3"/>
@@
 <junction x="17.78" y="172.72"/>
 <pinref part="IC2" gate="IC" pin="VOUT"/>
+<pinref part="C10" gate="G$1" pin="+"/>
 </segment>
 <segment>
@@
 <wire x1="-7.62" y1="160.02" x2="-22.86" y2="160.02" width="0.1524" layer="91"/>
 <wire x1="-22.86" y1="160.02" x2="-22.86" y2="162.56" width="0.1524" layer="91"/>
-<pinref part="C16" gate="G$1" pin="-"/>
 <wire x1="7.62" y1="160.02" x2="17.78" y2="160.02" width="0.1524" layer="91"/>
 <wire x1="17.78" y1="160.02" x2="17.78" y2="162.56" width="0.1524" layer="91"/>
 <junction x="7.62" y="160.02"/>
-<pinref part="C17" gate="G$1" pin="-"/>
 <wire x1="-22.86" y1="160.02" x2="-33.02" y2="160.02" width="0.1524" layer="91"/>
 <wire x1="-33.02" y1="160.02" x2="-33.02" y2="162.56" width="0.1524" layer="91"/>
 <junction x="-22.86" y="160.02"/>
 <pinref part="IC2" gate="IC" pin="GND"/>
+<pinref part="C9" gate="G$1" pin="-"/>
+<pinref part="C10" gate="G$1" pin="-"/>
 </segment>
 <segment>
@@
 <pinref part="P+2" gate="1" pin="+5V"/>
 <wire x1="-33.02" y1="172.72" x2="-33.02" y2="177.8" width="0.1524" layer="91"/>
-<pinref part="C17" gate="G$1" pin="+"/>
 <wire x1="-33.02" y1="172.72" x2="-33.02" y2="170.18" width="0.1524" layer="91"/>
 <junction x="-33.02" y="172.72"/>
 <pinref part="IC2" gate="IC" pin="VIN"/>
+<pinref part="C9" gate="G$1" pin="+"/>
 </segment>
 <segment>
@@
 </segment>
 <segment>
-<wire x1="157.48" y1="121.92" x2="160.02" y2="121.92" width="0.1524" layer="91"/>
-<label x="160.02" y="121.92" size="1.778" layer="95" xref="yes"/>
-<pinref part="IC1" gate="MCU" pin="PB12"/>
-</segment>
-</net>
+<wire x1="157.48" y1="93.98" x2="162.56" y2="93.98" width="0.1524" layer="91"/>
+<label x="162.56" y="93.98" size="1.778" layer="95" xref="yes"/>
+<pinref part="IC1" gate="MCU" pin="PB1"/>
+</segment>
+</net>

Commit message: final PCB corrections
Parts:
- added C11: 100n, resistormod:C-EUC0603K
- added PA0, PA1, PA2, PA3, PA4, PC0, PC1, PC2, PC3: (no value), wirepad:SMD2
- added R1, R5: 10k, resistor:R-EU_R0603
Connections:
- new net ADC_5V: C11.1, IC1MCU.PB0, R1.1, R5.2
- new net N$1: IC1MCU.PC0, PC0.P
- new net N$29: IC1MCU.PC1, PC1.P
- new net N$30: IC1MCU.PC2, PC2.P
- new net N$31: IC1MCU.PC3, PC3.P
- new net N$32: IC1MCU.PA0-WKUP, PA0.P
- new net N$37: IC1MCU.PA1, PA1.P
- new net N$41: IC1MCU.PA2, PA2.P
- new net N$45: IC1MCU.PA3, PA3.P
- new net N$65: IC1MCU.PA4, PA4.P
- net +5V: now also R1.2
- net GND: now also C11.2, R5.1
