File: hardware/batsim1_2.brd (EAGLE design)
At the start: 72 x 85 mm, 170 parts, among them IC1 OP07CR, IC10 MCP41HVX1, IC11 MCP47X6, IC12 L5973D, IC13 MAX44241, IC15 STM32F030C8T, IC16 TL084D, IC2 OP07CR, IC22 VREG-TS1117CW-5V, IC3 TL074D, IC4 DAC8552, IC5 DAC8552, IC6 LM334Z, IC7 TL084D, IC8 ADUM1301, IC9 LM2611, K1 G5LE, Q1 TIP2955, Q10 BC807-40SMD, Q11 BC817-40SMD, Q12 BC817-40SMD, Q13 BC817-40SMD, Q14 BC807-40SMD, Q2 TIP3055, Q3 TIP41C, Q4 TIP42C, Q5 BC807-40SMD, Q6 BC817-40SMD, Q7 BC817-40SMD, Q8 BC807-40SMD, Q9 BC807-40SMD

Commit message: board update
Connections:
- net N$15 renamed EXT_MISO
Changed lines of the file:
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@@
 <setting verticaltext="up"/>
 </settings>
-<grid distance="0.0125" unitdist="inch" unit="inch" style="lines" multiple="1" display="yes" altdistance="0.00625" altunitdist="inch" altunit="inch"/>
+<grid distance="0.1" unitdist="mm" unit="mm" style="lines" multiple="1" display="yes" altdistance="0.01" altunitdist="mm" altunit="mm"/>
 <layers>
 <layer number="1" name="Top" color="4" fill="1" visible="yes" active="yes"/>
@@
 <wire x1="46.51" y1="58.8925" x2="48.455" y2="58.8925" width="0.3048" layer="1"/>
 </signal>
-<signal name="N$15">
+<signal name="EXT_MISO">
 <contactref element="IC8" pad="12"/>
 <contactref element="IC15" pad="27"/>

Commit message: PCB markings
Connections:
- net N$32 renamed SWDIO
- net N$33 renamed SWCLK
- net N$34 renamed NRST
Other:
- board text added: "3V3"
- board text added: "5V"
- board text added: "Battery simulator"
- board text added: "GND"
- board text added: "MISO"
- board text added: "MOSI"
- board text added: "NRST"
- board text added: "OUT+"
- board text added: "OUT-"
- board text added: "SCK"
- board text added: "SWCLK"
- board text added: "SWDIO"
- board text added: "batsim V1.2 04/2017"
- board text added: "github.com/jankae/battery-sim"
Changed lines of the file:
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@@
 <setting verticaltext="up"/>
 </settings>
-<grid distance="0.1" unitdist="mm" unit="mm" style="lines" multiple="1" display="yes" altdistance="0.01" altunitdist="mm" altunit="mm"/>
+<grid distance="0.0125" unitdist="inch" unit="inch" style="lines" multiple="1" display="yes" altdistance="0.01" altunitdist="mm" altunit="mm"/>
 <layers>
 <layer number="1" name="Top" color="4" fill="1" visible="yes" active="yes"/>
@@
 <layer number="14" name="Route14" color="1" fill="6" visible="no" active="no"/>
 <layer number="15" name="Route15" color="4" fill="6" visible="no" active="no"/>
-<layer number="16" name="Bottom" color="1" fill="1" visible="yes" active="yes"/>
+<layer number="16" name="Bottom" color="1" fill="1" visible="no" active="yes"/>
 <layer number="17" name="Pads" color="2" fill="1" visible="yes" active="yes"/>
 <layer number="18" name="Vias" color="2" fill="1" visible="yes" active="yes"/>
@@
 <layer number="20" name="Dimension" color="15" fill="1" visible="yes" active="yes"/>
 <layer number="21" name="tPlace" color="7" fill="1" visible="yes" active="yes"/>
-<layer number="22" name="bPlace" color="7" fill="1" visible="yes" active="yes"/>
+<layer number="22" name="bPlace" color="7" fill="1" visible="no" active="yes"/>
 <layer number="23" name="tOrigins" color="15" fill="1" visible="yes" active="yes"/>
-<layer number="24" name="bOrigins" color="15" fill="1" visible="yes" active="yes"/>
+<layer number="24" name="bOrigins" color="15" fill="1" visible="no" active="yes"/>
 <layer number="25" name="tNames" color="7" fill="1" visible="no" active="yes"/>
 <layer number="26" name="bNames" color="7" fill="1" visible="no" active="yes"/>
@@
 <layer number="38" name="bTest" color="7" fill="1" visible="no" active="yes"/>
 <layer number="39" name="tKeepout" color="4" fill="11" visible="yes" active="yes"/>
-<layer number="40" name="bKeepout" color="1" fill="11" visible="yes" active="yes"/>
+<layer number="40" name="bKeepout" color="1" fill="11" visible="no" active="yes"/>
 <layer number="41" name="tRestrict" color="4" fill="10" visible="yes" active="yes"/>
-<layer number="42" name="bRestrict" color="1" fill="10" visible="yes" active="yes"/>
+<layer number="42" name="bRestrict" color="1" fill="10" visible="no" active="yes"/>
 <layer number="43" name="vRestrict" color="2" fill="10" visible="no" active="yes"/>
 <layer number="44" name="Drills" color="7" fill="1" visible="no" active="yes"/>
@@
 <layer number="50" name="dxf" color="7" fill="1" visible="no" active="no"/>
 <layer number="51" name="tDocu" color="7" fill="1" visible="yes" active="yes"/>
-<layer number="52" name="bDocu" color="7" fill="1" visible="yes" active="yes"/>
+<layer number="52" name="bDocu" color="7" fill="1" visible="no" active="yes"/>
 <layer number="53" name="tGND_GNDA" color="7" fill="9" visible="no" active="no"/>
 <layer number="54" name="bGND_GNDA" color="1" fill="9" visible="no" active="no"/>
@@
 <layer number="118" name="Rect_Pads" color="4" fill="1" visible="no" active="yes"/>
 <layer number="121" name="_tsilk" color="7" fill="1" visible="yes" active="yes"/>
-<layer number="122" name="_bsilk" color="7" fill="1" visible="yes" active="yes"/>
+<layer number="122" name="_bsilk" color="7" fill="1" visible="no" active="yes"/>
 <layer number="123" name="tTestmark" color="7" fill="1" visible="no" active="yes"/>
 <layer number="124" name="bTestmark" color="7" fill="1" visible="no" active="yes"/>
@@
 <rectangle x1="37.1475" y1="21.59" x2="40.3225" y2="25.4" layer="42"/>
 <rectangle x1="64.135" y1="20.32" x2="66.675" y2="26.035" layer="41"/>
+<text x="48.4" y="82.5" size="1.016" layer="21" font="vector">GND</text>
+<text x="50.8" y="83.7" size="1.016" layer="21" font="vector">MISO</text>
+<text x="53.5" y="82.5" size="1.016" layer="21" font="vector">SCK</text>
+<text x="55.8" y="83.7" size="1.016" layer="21" font="vector">MOSI</text>
+<text x="58.6" y="82.5" size="1.016" layer="21" font="vector">3V3</text>
+<text x="61.6" y="83.7" size="1.016" layer="21" font="vector">5V</text>
+<text x="14.4" y="82.5" size="2.1844" layer="21" font="vector">OUT-</text>
+<text x="24.6" y="82.5" size="2.1844" layer="21" font="vector">OUT+</text>
+<text x="46" y="80.6" size="0.8128" layer="21" font="vector" rot="R90">3V3</text>
+<text x="41.7" y="77.4" size="0.8128" layer="21" font="vector" rot="R90">SWCLK</text>
+<text x="46" y="75.5" size="0.8128" layer="21" font="vector" rot="R90">GND</text>
+<text x="41.8" y="72.3" size="0.8128" layer="21" font="vector" rot="R90">SWDIO</text>
+<text x="46.1" y="70.1" size="0.8128" layer="21" font="vector" rot="R90">NRST</text>
+<text x="59.69" y="11.7475" size="3.81" layer="22" font="vector" rot="MR90">Battery simulator</text>
+<text x="53.975" y="11.7475" size="2.54" layer="22" font="vector" rot="MR90">batsim V1.2   04/2017</text>
+<text x="50.8" y="11.7475" size="2.1844" layer="22" font="vector" rot="MR90">github.com/jankae/battery-sim</text>
 </plain>
 <attributes>
@@
 <attribute name="VALUE" x="68.58" y="55.753" size="0.0254" layer="27"/>
 </element>
-<element name="BAT_OUT" library="pinhead" package="1X08/90" value="" x="23.09" y="84.65" locked="yes" rot="MR0"/>
+<element name="BAT_OUT" library="pinhead" package="1X08/90" value="" x="23.09" y="84.65" locked="yes" smashed="yes" rot="MR0">
+<attribute name="VALUE" x="11.025" y="80.84" size="1.27" layer="28" rot="MR90"/>
+</element>
 <element name="C1" library="rcl" package="C1206" value="22u/16V" x="42.8625" y="22.225" smashed="yes" rot="R180">
 <attribute name="NAME" x="45.085" y="22.5425" size="0.8128" layer="25" font="vector" rot="R270"/>
@@
 <attribute name="VALUE" x="36.8225" y="30.69" size="1.016" layer="27" ratio="18" rot="R270"/>
 </element>
-<element name="FRONTPANEL" library="pinhead" package="1X06/90" value="" x="56.11" y="84.65" locked="yes" rot="MR0"/>
+<element name="FRONTPANEL" library="pinhead" package="1X06/90" value="" x="56.11" y="84.65" locked="yes" smashed="yes" rot="MR0">
+<attribute name="VALUE" x="46.585" y="80.84" size="1.27" layer="28" rot="MR90"/>
+</element>
 <element name="IC1" library="linear" package="SO08" value="OP07CR" x="42.2275" y="39.6875" smashed="yes">
 <attribute name="NAME" x="39.5605" y="41.5925" size="0.8128" layer="25" font="vector" rot="R90"/>
@@
 </element>
 <element name="SDIO" library="pinhead" package="1X05" value="" x="43.4975" y="76.5175" smashed="yes" rot="R270">
-<attribute name="NAME" x="45.3263" y="82.9437" size="0.8128" layer="25" font="vector" ratio="10" rot="R270"/>
+<attribute name="NAME" x="42.2563" y="83.2263" size="0.8128" layer="25" font="vector" ratio="10"/>
 <attribute name="VALUE" x="40.3225" y="82.8675" size="1.27" layer="27" rot="R270"/>
 </element>
@@
 <vertex x="61.9125" y="28.575"/>
 <vertex x="72.7075" y="28.575"/>
-<vertex x="72.7075" y="71.755"/>
+<vertex x="72.7075" y="67.655"/>
+<vertex x="71.045" y="69.155"/>
+<vertex x="68.4" y="71.8"/>
 <vertex x="48.26" y="71.755"/>
 <vertex x="46.6725" y="73.3425"/>
-<vertex x="46.6725" y="85.4075"/>
+<vertex x="46.4" y="81.9"/>
+<vertex x="43.3725" y="84.9275"/>
+<vertex x="42.8725" y="85.4075"/>
 </polygon>
 <wire x1="51.1175" y1="20.32" x2="51.1175" y2="19.18" width="0.4064" layer="16"/>
@@
 <wire x1="56.1975" y1="66.51625" x2="56.1975" y2="67.79" width="0.3048" layer="1"/>
 </signal>
-<signal name="N$32">
+<signal name="SWDIO">
 <contactref element="IC15" pad="34"/>
 <contactref element="SDIO" pad="4"/>
@@
 <wire x1="44.45" y1="73.9775" x2="43.4975" y2="73.9775" width="0.3048" layer="1"/>
 </signal>
-<signal name="N$33">
+<signal name="SWCLK">
 <contactref element="IC15" pad="37"/>
 <contactref element="SDIO" pad="2"/>
@@
 <wire x1="41.5925" y1="77.1525" x2="43.4975" y2="79.0575" width="0.3048" layer="1"/>
 </signal>
-<signal name="N$34">
+<signal name="NRST">
 <contactref element="SDIO" pad="5"/>
 <contactref element="IC15" pad="7"/>

Commit message: minor PCB changes
Parts:
- D8: value (none) -> SS110
- moved R10 5.08 mm to (4.76, 35.9), turned to 270 degrees
- moved R11 3.19 mm to (2.22, 36.5), turned to 0 degrees
- moved IC13 2.29 mm to (3.81, 40.3), turned to 0 degrees
- moved C18 1.59 mm to (5.40, 32.1), turned to 0 degrees
- moved C19 0.63 mm to (2.22, 34.3)
- moved R35 0.63 mm to (2.22, 32.1)
Connections:
- new net N$15: IC3.6, IC3.7
- new net N$27: IC16.13, IC16.14
- net +3V3: now also IC8.10
- net GND: now also IC16.12, IC3.5
- net N$45: now also IC8.7
Routing:
- net GND: track 695.0 -> 708.4 mm, vias 140 -> 142
- net N$45: track 4.34 -> 13.7 mm, vias 0 -> 2
- net +3V3: track 188.8 -> 196.6 mm, vias 14 -> 15
- net +24V: track 249.4 -> 244.6 mm
- net CURRENT_SENSE: track 98.5 -> 103.1 mm
- net N$5: track 83.4 -> 78.9 mm
- net N$14: track 7.96 -> 3.58 mm
- net BATTERY+: track 44.8 -> 40.8 mm
- net -8V: track 158.5 -> 156.1 mm
- net N$39: track 6.38 -> 8.33 mm
- net N$38: track 22.3 -> 20.8 mm
- net N$27: track 0.00 -> 1.27 mm
- net N$15: track 0.00 -> 1.27 mm
- net N$22: track 23.5 -> 22.4 mm

Commit message: Minor hardware + gitignore update
Parts:
- C19: value 200p -> 100p
- C28: value 100n -> 10u/35V
- C5: value 100p -> 330p
- R12: value 10k -> n.p.
- R2, R6: value 1k5 -> 3k3
- R31: value 10k -> 1k
- R44: value 10k -> 5k
- R51: value 100k -> 47k
Changed lines of the file:
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@@
 <setting verticaltext="up"/>
 </settings>
-<grid distance="0.0125" unitdist="inch" unit="inch" style="lines" multiple="1" display="yes" altdistance="0.00625" altunitdist="inch" altunit="inch"/>
+<grid distance="0.0125" unitdist="inch" unit="mm" style="lines" multiple="1" display="yes" altdistance="0.00625" altunitdist="inch" altunit="inch"/>
 <layers>
 <layer number="1" name="Top" color="4" fill="1" visible="yes" active="yes"/>
@@
 <layer number="14" name="Route14" color="1" fill="6" visible="no" active="no"/>
 <layer number="15" name="Route15" color="4" fill="6" visible="no" active="no"/>
-<layer number="16" name="Bottom" color="1" fill="1" visible="no" active="yes"/>
+<layer number="16" name="Bottom" color="1" fill="1" visible="yes" active="yes"/>
 <layer number="17" name="Pads" color="2" fill="1" visible="yes" active="yes"/>
 <layer number="18" name="Vias" color="2" fill="1" visible="yes" active="yes"/>
@@
 <layer number="20" name="Dimension" color="15" fill="1" visible="yes" active="yes"/>
 <layer number="21" name="tPlace" color="7" fill="1" visible="yes" active="yes"/>
-<layer number="22" name="bPlace" color="7" fill="1" visible="no" active="yes"/>
+<layer number="22" name="bPlace" color="7" fill="1" visible="yes" active="yes"/>
 <layer number="23" name="tOrigins" color="15" fill="1" visible="yes" active="yes"/>
-<layer number="24" name="bOrigins" color="15" fill="1" visible="no" active="yes"/>
+<layer number="24" name="bOrigins" color="15" fill="1" visible="yes" active="yes"/>
 <layer number="25" name="tNames" color="7" fill="1" visible="no" active="yes"/>
 <layer number="26" name="bNames" color="7" fill="1" visible="no" active="yes"/>
@@
 <layer number="38" name="bTest" color="7" fill="1" visible="no" active="yes"/>
 <layer number="39" name="tKeepout" color="4" fill="11" visible="yes" active="yes"/>
-<layer number="40" name="bKeepout" color="1" fill="11" visible="no" active="yes"/>
+<layer number="40" name="bKeepout" color="1" fill="11" visible="yes" active="yes"/>
 <layer number="41" name="tRestrict" color="4" fill="10" visible="yes" active="yes"/>
-<layer number="42" name="bRestrict" color="1" fill="10" visible="no" active="yes"/>
+<layer number="42" name="bRestrict" color="1" fill="10" visible="yes" active="yes"/>
 <layer number="43" name="vRestrict" color="2" fill="10" visible="no" active="yes"/>
 <layer number="44" name="Drills" color="7" fill="1" visible="no" active="yes"/>
@@
 <layer number="50" name="dxf" color="7" fill="1" visible="no" active="no"/>
 <layer number="51" name="tDocu" color="7" fill="1" visible="yes" active="yes"/>
-<layer number="52" name="bDocu" color="7" fill="1" visible="no" active="yes"/>
+<layer number="52" name="bDocu" color="7" fill="1" visible="yes" active="yes"/>
 <layer number="53" name="tGND_GNDA" color="7" fill="9" visible="no" active="no"/>
 <layer number="54" name="bGND_GNDA" color="1" fill="9" visible="no" active="no"/>
@@
 <layer number="118" name="Rect_Pads" color="4" fill="1" visible="no" active="yes"/>
 <layer number="121" name="_tsilk" color="7" fill="1" visible="yes" active="yes"/>
-<layer number="122" name="_bsilk" color="7" fill="1" visible="no" active="yes"/>
+<layer number="122" name="_bsilk" color="7" fill="1" visible="yes" active="yes"/>
 <layer number="123" name="tTestmark" color="7" fill="1" visible="no" active="yes"/>
 <layer number="124" name="bTestmark" color="7" fill="1" visible="no" active="yes"/>
@@
 <attribute name="VALUE" x="4.7625" y="30.1625" size="1.27" layer="27"/>
 </element>
-<element name="C19" library="rcl" package="C0603" value="200p" x="2.2225" y="34.29" smashed="yes" rot="R180">
+<element name="C19" library="rcl" package="C0603" value="100p" x="2.2225" y="34.29" smashed="yes" rot="R180">
 <attribute name="NAME" x="3.175" y="33.655" size="0.8128" layer="25" font="vector" rot="R180"/>
 <attribute name="VALUE" x="2.8575" y="36.195" size="1.27" layer="27" rot="R180"/>
@@
 <attribute name="VALUE" x="64.4525" y="58.7375" size="1.27" layer="27" rot="R90"/>
 </element>
-<element name="C28" library="rcl" package="C1206" value="100n" x="20.32" y="45.72" smashed="yes" rot="R90">
+<element name="C28" library="rcl" package="C1206" value="10u/35V" x="20.32" y="45.72" smashed="yes" rot="R90">
 <attribute name="NAME" x="22.225" y="46.6725" size="0.8128" layer="25" font="vector" rot="R90"/>
 <attribute name="VALUE" x="22.86" y="44.45" size="1.27" layer="27" rot="R90"/>
@@
 <attribute name="VALUE" x="38.4175" y="75.8825" size="1.27" layer="27"/>
 </element>
-<element name="C5" library="rcl" package="C0603" value="100p" x="12.7" y="22.225" smashed="yes" rot="R270">
+<element name="C5" library="rcl" package="C0603" value="330p" x="12.7" y="22.225" smashed="yes" rot="R270">
 <attribute name="NAME" x="14.2875" y="21.59" size="0.8128" layer="25" font="vector" rot="R90"/>
 <attribute name="VALUE" x="10.795" y="22.86" size="1.27" layer="27" rot="R270"/>
@@
 <attribute name="VALUE" x="1.5875" y="34.6075" size="1.27" layer="27"/>
 </element>
-<element name="R12" library="resistor" package="R0603" value="10k" x="19.3675" y="22.5425" smashed="yes" rot="R90">
+<element name="R12" library="resistor" package="R0603" value="n.p." x="19.3675" y="22.5425" smashed="yes" rot="R90">
 <attribute name="NAME" x="21.2725" y="21.59" size="0.8128" layer="25" font="vector" rot="R90"/>
 <attribute name="VALUE" x="21.2725" y="21.9075" size="1.27" layer="27" rot="R90"/>
@@
 <attribute name="VALUE" x="40.48125" y="39.0525" size="1.27" layer="27" rot="R90"/>
 </element>
-<element name="R2" library="resistor" package="R0603" value="1k5" x="61.9125" y="5.715" smashed="yes" rot="R90">
+<element name="R2" library="resistor" package="R0603" value="3k3" x="61.9125" y="5.715" smashed="yes" rot="R90">
 <attribute name="NAME" x="61.2775" y="5.08" size="0.8128" layer="25" font="vector" rot="R90"/>
 <attribute name="VALUE" x="63.8175" y="5.08" size="1.27" layer="27" rot="R90"/>
@@
 <attribute name="VALUE" x="10.795" y="29.845" size="1.27" layer="27" rot="R270"/>
 </element>
-<element name="R31" library="resistor" package="R0603" value="10k" x="42.2275" y="61.2775" smashed="yes" rot="R270">
+<element name="R31" library="resistor" package="R0603" value="1k" x="42.2275" y="61.2775" smashed="yes" rot="R270">
 <attribute name="NAME" x="42.8625" y="61.9125" size="0.8128" layer="25" font="vector" rot="R270"/>
 <attribute name="VALUE" x="40.3225" y="61.9125" size="1.27" layer="27" rot="R270"/>
@@
 <attribute name="VALUE" x="54.9275" y="46.6725" size="1.27" layer="27" rot="R90"/>
 </element>
-<element name="R44" library="resistor" package="R0603" value="10k" x="14.9225" y="22.5425" smashed="yes" rot="R270">
+<element name="R44" library="resistor" package="R0603" value="5k" x="14.9225" y="22.5425" smashed="yes" rot="R270">
 <attribute name="NAME" x="16.51" y="21.59" size="0.8128" layer="25" font="vector" rot="R90"/>
 <attribute name="VALUE" x="13.0175" y="23.1775" size="1.27" layer="27" rot="R270"/>
@@
 <attribute name="VALUE" x="66.9925" y="48.26" size="1.27" layer="27" rot="R90"/>
 </element>
-<element name="R51" library="resistor" package="R0603" value="100k" x="55.5625" y="37.1475" smashed="yes" rot="R270">
+<element name="R51" library="resistor" package="R0603" value="47k" x="55.5625" y="37.1475" smashed="yes" rot="R270">
 <attribute name="NAME" x="53.975" y="39.0525" size="0.8128" layer="25" font="vector" rot="R270"/>
 <attribute name="VALUE" x="53.6575" y="37.7825" size="1.27" layer="27" rot="R270"/>
@@
 <attribute name="VALUE" x="64.61125" y="60.0075" size="1.27" layer="27" rot="R270"/>
 </element>
-<element name="R6" library="resistor" package="R0603" value="1k5" x="10.16" y="5.08" smashed="yes" rot="R180">
+<element name="R6" library="resistor" package="R0603" value="3k3" x="10.16" y="5.08" smashed="yes" rot="R180">
 <attribute name="NAME" x="10.795" y="6.6675" size="0.8128" layer="25" font="vector" rot="R180"/>
 <attribute name="VALUE" x="10.795" y="6.985" size="1.27" layer="27" rot="R180"/>
