File: hardware/batsim1_2.sch (EAGLE design)
At the start: 170 parts, among them IC1 OP07CR, IC10 MCP41HVX1, IC11 MCP47X6, IC12 L5973D, IC13 MAX44241, IC15 STM32F030C8T, IC16 TL084D, IC2 OP07CR, IC22 VREG-TS1117CW-5V, IC3 TL074D, IC4 DAC8552, IC5 DAC8552, IC6 LM334Z, IC7 TL084D, IC8 ADUM1301, IC9 LM2611, K1 G5LE, Q1 TIP2955, Q10 BC807-40SMD, Q11 BC817-40SMD, Q12 BC817-40SMD, Q13 BC817-40SMD, Q14 BC807-40SMD, Q2 TIP3055, Q3 TIP41C, Q4 TIP42C, Q5 BC807-40SMD, Q6 BC817-40SMD, Q7 BC817-40SMD, Q8 BC807-40SMD, Q9 BC807-40SMD

Commit message: board update
Connections:
- net N$15 renamed EXT_MISO
Changed lines of the file:
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@@
 <grid distance="0.1" unitdist="inch" unit="inch" style="lines" multiple="1" display="no" altdistance="0.01" altunitdist="inch" altunit="inch"/>
 <layers>
-<layer number="1" name="Top" color="4" fill="1" visible="yes" active="no"/>
-<layer number="2" name="Route2" color="1" fill="3" visible="yes" active="no"/>
-<layer number="3" name="Route3" color="4" fill="3" visible="yes" active="no"/>
-<layer number="14" name="Route14" color="1" fill="6" visible="yes" active="no"/>
-<layer number="15" name="Route15" color="4" fill="6" visible="yes" active="no"/>
-<layer number="16" name="Bottom" color="1" fill="1" visible="yes" active="no"/>
-<layer number="17" name="Pads" color="2" fill="1" visible="yes" active="no"/>
-<layer number="18" name="Vias" color="2" fill="1" visible="yes" active="no"/>
-<layer number="19" name="Unrouted" color="6" fill="1" visible="yes" active="no"/>
-<layer number="20" name="Dimension" color="15" fill="1" visible="yes" active="no"/>
-<layer number="21" name="tPlace" color="7" fill="1" visible="yes" active="no"/>
-<layer number="22" name="bPlace" color="7" fill="1" visible="yes" active="no"/>
-<layer number="23" name="tOrigins" color="15" fill="1" visible="yes" active="no"/>
-<layer number="24" name="bOrigins" color="15" fill="1" visible="yes" active="no"/>
-<layer number="25" name="tNames" color="7" fill="1" visible="yes" active="no"/>
-<layer number="26" name="bNames" color="7" fill="1" visible="yes" active="no"/>
-<layer number="27" name="tValues" color="7" fill="1" visible="yes" active="no"/>
-<layer number="28" name="bValues" color="7" fill="1" visible="yes" active="no"/>
+<layer number="1" name="Top" color="4" fill="1" visible="no" active="no"/>
+<layer number="2" name="Route2" color="1" fill="3" visible="no" active="no"/>
+<layer number="3" name="Route3" color="4" fill="3" visible="no" active="no"/>
+<layer number="14" name="Route14" color="1" fill="6" visible="no" active="no"/>
+<layer number="15" name="Route15" color="4" fill="6" visible="no" active="no"/>
+<layer number="16" name="Bottom" color="1" fill="1" visible="no" active="no"/>
+<layer number="17" name="Pads" color="2" fill="1" visible="no" active="no"/>
+<layer number="18" name="Vias" color="2" fill="1" visible="no" active="no"/>
+<layer number="19" name="Unrouted" color="6" fill="1" visible="no" active="no"/>
+<layer number="20" name="Dimension" color="15" fill="1" visible="no" active="no"/>
+<layer number="21" name="tPlace" color="7" fill="1" visible="no" active="no"/>
+<layer number="22" name="bPlace" color="7" fill="1" visible="no" active="no"/>
+<layer number="23" name="tOrigins" color="15" fill="1" visible="no" active="no"/>
+<layer number="24" name="bOrigins" color="15" fill="1" visible="no" active="no"/>
+<layer number="25" name="tNames" color="7" fill="1" visible="no" active="no"/>
+<layer number="26" name="bNames" color="7" fill="1" visible="no" active="no"/>
+<layer number="27" name="tValues" color="7" fill="1" visible="no" active="no"/>
+<layer number="28" name="bValues" color="7" fill="1" visible="no" active="no"/>
 <layer number="29" name="tStop" color="7" fill="3" visible="no" active="no"/>
 <layer number="30" name="bStop" color="7" fill="6" visible="no" active="no"/>
@@
 <layer number="35" name="tGlue" color="7" fill="4" visible="no" active="no"/>
 <layer number="36" name="bGlue" color="7" fill="5" visible="no" active="no"/>
-<layer number="37" name="tTest" color="7" fill="1" visible="yes" active="no"/>
-<layer number="38" name="bTest" color="7" fill="1" visible="yes" active="no"/>
+<layer number="37" name="tTest" color="7" fill="1" visible="no" active="no"/>
+<layer number="38" name="bTest" color="7" fill="1" visible="no" active="no"/>
 <layer number="39" name="tKeepout" color="4" fill="11" visible="no" active="no"/>
 <layer number="40" name="bKeepout" color="1" fill="11" visible="no" active="no"/>
@@
 <layer number="44" name="Drills" color="7" fill="1" visible="no" active="no"/>
 <layer number="45" name="Holes" color="7" fill="1" visible="no" active="no"/>
-<layer number="46" name="Milling" color="3" fill="1" visible="yes" active="no"/>
-<layer number="47" name="Measures" color="7" fill="1" visible="yes" active="no"/>
-<layer number="48" name="Document" color="7" fill="1" visible="yes" active="no"/>
-<layer number="49" name="Reference" color="7" fill="1" visible="yes" active="no"/>
-<layer number="50" name="dxf" color="7" fill="1" visible="yes" active="no"/>
-<layer number="51" name="tDocu" color="7" fill="1" visible="yes" active="no"/>
-<layer number="52" name="bDocu" color="7" fill="1" visible="yes" active="no"/>
-<layer number="53" name="tGND_GNDA" color="7" fill="9" visible="yes" active="no"/>
-<layer number="54" name="bGND_GNDA" color="1" fill="9" visible="yes" active="no"/>
-<layer number="56" name="wert" color="7" fill="1" visible="yes" active="no"/>
+<layer number="46" name="Milling" color="3" fill="1" visible="no" active="no"/>
+<layer number="47" name="Measures" color="7" fill="1" visible="no" active="no"/>
+<layer number="48" name="Document" color="7" fill="1" visible="no" active="no"/>
+<layer number="49" name="Reference" color="7" fill="1" visible="no" active="no"/>
+<layer number="50" name="dxf" color="7" fill="1" visible="no" active="no"/>
+<layer number="51" name="tDocu" color="7" fill="1" visible="no" active="no"/>
+<layer number="52" name="bDocu" color="7" fill="1" visible="no" active="no"/>
+<layer number="53" name="tGND_GNDA" color="7" fill="9" visible="no" active="no"/>
+<layer number="54" name="bGND_GNDA" color="1" fill="9" visible="no" active="no"/>
+<layer number="56" name="wert" color="7" fill="1" visible="no" active="no"/>
 <layer number="90" name="Modules" color="5" fill="1" visible="yes" active="yes"/>
 <layer number="91" name="Nets" color="2" fill="1" visible="yes" active="yes"/>
@@
 </segment>
 </net>
-<net name="N$15" class="0">
+<net name="EXT_MISO" class="0">
 <segment>
 <pinref part="IC8" gate="G$1" pin="VIC"/>

Commit message: PCB markings
Connections:
- net N$32 renamed SWDIO
- net N$33 renamed SWCLK
- net N$34 renamed NRST
Changed lines of the file:
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@@
 </segment>
 </net>
-<net name="N$32" class="0">
+<net name="SWDIO" class="0">
 <segment>
 <pinref part="IC15" gate="MCU" pin="PA13"/>
@@
 </segment>
 </net>
-<net name="N$33" class="0">
+<net name="SWCLK" class="0">
 <segment>
 <pinref part="IC15" gate="MCU" pin="PA14"/>
@@
 </segment>
 </net>
-<net name="N$34" class="0">
+<net name="NRST" class="0">
 <segment>
 <pinref part="SDIO" gate="A" pin="5"/>

Commit message: minor PCB changes
Parts:
- D8: value (none) -> SS110
Connections:
- new net N$15: IC3B.-IN, IC3B.OUT
- new net N$27: IC16D.-IN, IC16D.OUT
- net +3V3: now also IC8.VE2
- net GND: now also IC16D.+IN, IC3B.+IN
- net N$45: now also IC8.VE1
Other:
- moved on the sheet: IC16D, IC3B
Changed lines of the file:
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@@
 <part name="C37" library="rcl" deviceset="C-EU" device="C1206" value="1u/25V"/>
 <part name="SUPPLY9" library="supply2" deviceset="-8V" device=""/>
-<part name="D8" library="diodes" deviceset="D-" device="SMA"/>
+<part name="D8" library="diodes" deviceset="D-" device="SMA" value="SS110"/>
 <part name="GND41" library="supply1" deviceset="GND" device=""/>
 <part name="R55" library="resistor" deviceset="R-EU_" device="R0603" value="9k1"/>
@@
 <part name="GND59" library="supply1" deviceset="GND" device=""/>
 <part name="P+16" library="supply1" deviceset="+24V" device=""/>
+<part name="GND60" library="supply1" deviceset="GND" device=""/>
+<part name="GND61" library="supply1" deviceset="GND" device=""/>
 </parts>
 <sheets>
@@
 <instance part="+3V6" gate="G$1" x="287.02" y="96.52"/>
 <instance part="GND6" gate="1" x="396.24" y="81.28"/>
-<instance part="+3V8" gate="G$1" x="396.24" y="109.22"/>
+<instance part="+3V8" gate="G$1" x="393.7" y="109.22"/>
 <instance part="SUPPLY10" gate="G$1" x="439.42" y="109.22"/>
 <instance part="SUPPLY11" gate="G$1" x="431.8" y="81.28"/>
@@
 <instance part="IC16" gate="C" x="467.36" y="269.24" rot="MR180"/>
 <instance part="IC16" gate="B" x="497.84" y="236.22" rot="MR180"/>
-<instance part="IC3" gate="B" x="444.5" y="205.74"/>
-<instance part="IC16" gate="D" x="469.9" y="205.74"/>
+<instance part="IC3" gate="B" x="449.58" y="205.74"/>
+<instance part="IC16" gate="D" x="474.98" y="205.74"/>
 <instance part="IC16" gate="P" x="403.86" y="347.98"/>
 <instance part="R46" gate="G$1" x="449.58" y="271.78" smashed="yes">
@@
 <instance part="C30" gate="G$1" x="114.3" y="347.98" rot="MR180"/>
 <instance part="IC22" gate="IC" x="152.4" y="309.88"/>
+<instance part="GND60" gate="1" x="436.88" y="208.28" rot="R270"/>
+<instance part="GND61" gate="1" x="462.28" y="208.28" rot="R270"/>
 </instances>
 <busses>
@@
 <pinref part="GND14" gate="1" pin="GND"/>
 <wire x1="241.3" y1="340.36" x2="241.3" y2="337.82" width="0.1524" layer="91"/>
+</segment>
+<segment>
+<pinref part="GND61" gate="1" pin="GND"/>
+<pinref part="IC16" gate="D" pin="+IN"/>
+<wire x1="464.82" y1="208.28" x2="467.36" y2="208.28" width="0.1524" layer="91"/>
+</segment>
+<segment>
+<pinref part="GND60" gate="1" pin="GND"/>
+<pinref part="IC3" gate="B" pin="+IN"/>
+<wire x1="439.42" y1="208.28" x2="441.96" y2="208.28" width="0.1524" layer="91"/>
 </segment>
 </net>
@@
 <pinref part="IC8" gate="G$1" pin="VDD2"/>
 <pinref part="+3V8" gate="G$1" pin="+3V3"/>
-<wire x1="398.78" y1="104.14" x2="396.24" y2="104.14" width="0.1524" layer="91"/>
-<wire x1="396.24" y1="104.14" x2="396.24" y2="106.68" width="0.1524" layer="91"/>
+<wire x1="398.78" y1="104.14" x2="393.7" y2="104.14" width="0.1524" layer="91"/>
+<wire x1="393.7" y1="104.14" x2="393.7" y2="106.68" width="0.1524" layer="91"/>
+<pinref part="IC8" gate="G$1" pin="VE2"/>
+<wire x1="398.78" y1="88.9" x2="393.7" y2="88.9" width="0.1524" layer="91"/>
+<wire x1="393.7" y1="88.9" x2="393.7" y2="104.14" width="0.1524" layer="91"/>
+<junction x="393.7" y="104.14"/>
 </segment>
 <segment>
@@
 <wire x1="434.34" y1="101.6" x2="434.34" y2="104.14" width="0.1524" layer="91"/>
 <wire x1="434.34" y1="104.14" x2="429.26" y2="104.14" width="0.1524" layer="91"/>
+<pinref part="IC8" gate="G$1" pin="VE1"/>
+<wire x1="429.26" y1="88.9" x2="434.34" y2="88.9" width="0.1524" layer="91"/>
+<wire x1="434.34" y1="88.9" x2="434.34" y2="101.6" width="0.1524" layer="91"/>
+<junction x="434.34" y="101.6"/>
 </segment>
 </net>
@@
 </segment>
 </net>
+<net name="N$15" class="0">
+<segment>
+<pinref part="IC3" gate="B" pin="OUT"/>
+<wire x1="457.2" y1="205.74" x2="459.74" y2="205.74" width="0.1524" layer="91"/>
+<wire x1="459.74" y1="205.74" x2="459.74" y2="198.12" width="0.1524" layer="91"/>
+<wire x1="459.74" y1="198.12" x2="439.42" y2="198.12" width="0.1524" layer="91"/>
+<wire x1="439.42" y1="198.12" x2="439.42" y2="203.2" width="0.1524" layer="91"/>
+<pinref part="IC3" gate="B" pin="-IN"/>
+<wire x1="439.42" y1="203.2" x2="441.96" y2="203.2" width="0.1524" layer="91"/>
+</segment>
+</net>
+<net name="N$27" class="0">
+<segment>
+<pinref part="IC16" gate="D" pin="OUT"/>
+<wire x1="482.6" y1="205.74" x2="485.14" y2="205.74" width="0.1524" layer="91"/>
+<wire x1="485.14" y1="205.74" x2="485.14" y2="198.12" width="0.1524" layer="91"/>
+<wire x1="485.14" y1="198.12" x2="464.82" y2="198.12" width="0.1524" layer="91"/>
+<wire x1="464.82" y1="198.12" x2="464.82" y2="203.2" width="0.1524" layer="91"/>
+<pinref part="IC16" gate="D" pin="-IN"/>
+<wire x1="464.82" y1="203.2" x2="467.36" y2="203.2" width="0.1524" layer="91"/>
+</segment>
+</net>
 </nets>
 </sheet>
 </sheets>
+<errors>
+</errors>
 </schematic>
 </drawing>

Commit message: Minor hardware + gitignore update
Parts:
- C19: value 200p -> 100p
- C28: value 100n -> 10u/35V
- C5: value 100p -> 330p
- R12: value 10k -> n.p.
- R2, R6: value 1k5 -> 3k3
- R31: value 10k -> 1k
- R44: value 10k -> 5k
- R51: value 100k -> 47k
Changed lines of the file:
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@@
 <part name="Q6" library="transistor-npn" deviceset="BC817*" device="SMD" technology="-40"/>
 <part name="R1" library="resistor" deviceset="R-EU_" device="R0603" value="100"/>
-<part name="R2" library="resistor" deviceset="R-EU_" device="R0603" value="1k5"/>
+<part name="R2" library="resistor" deviceset="R-EU_" device="R0603" value="3k3"/>
 <part name="R3" library="resistormod" deviceset="5WAXIAL" device="" value="0.1/5W"/>
 <part name="R4" library="resistormod" deviceset="5WAXIAL" device="" value="0.1/5W"/>
 <part name="R5" library="resistor" deviceset="R-EU_" device="R0603" value="100"/>
-<part name="R6" library="resistor" deviceset="R-EU_" device="R0603" value="1k5"/>
+<part name="R6" library="resistor" deviceset="R-EU_" device="R0603" value="3k3"/>
 <part name="Q7" library="transistor-npn" deviceset="BC817*" device="SMD" technology="-40"/>
 <part name="Q8" library="transistor-pnp" deviceset="BC807*" device="SMD" technology="-40"/>
@@
 <part name="R28" library="resistor" deviceset="R-EU_" device="R0603" value="1k"/>
 <part name="D3" library="zetex" deviceset="D" device="SOD323" value="1N4148"/>
-<part name="C5" library="rcl" deviceset="C-EU" device="C0603" value="100p"/>
+<part name="C5" library="rcl" deviceset="C-EU" device="C0603" value="330p"/>
 <part name="R29" library="resistor" deviceset="R-EU_" device="R0603" value="10k"/>
 <part name="K1" library="relay" deviceset="G5LE" device=""/>
@@
 <part name="GND15" library="supply1" deviceset="GND" device=""/>
 <part name="D4" library="zetex" deviceset="D" device="SOD323" value="1N4148"/>
-<part name="R31" library="resistor" deviceset="R-EU_" device="R0603" value="10k"/>
+<part name="R31" library="resistor" deviceset="R-EU_" device="R0603" value="1k"/>
 <part name="IC7" library="linear" deviceset="TL084" device="D"/>
 <part name="R33" library="resistor" deviceset="R-EU_" device="R0603" value="33k"/>
@@
 <part name="D5" library="zetex" deviceset="D" device="SOD323" value="1N4148"/>
 <part name="C18" library="rcl" deviceset="C-EU" device="C0603" value="10n"/>
-<part name="C19" library="rcl" deviceset="C-EU" device="C0603" value="200p"/>
+<part name="C19" library="rcl" deviceset="C-EU" device="C0603" value="100p"/>
 <part name="R35" library="resistor" deviceset="R-EU_" device="R0603" value="1k"/>
 <part name="Q14" library="transistor-pnp" deviceset="BC807*" device="SMD" technology="-40"/>
@@
 <part name="R36" library="resistor" deviceset="R-EU_" device="R0603" value="1k"/>
 <part name="FRAME1" library="frames" deviceset="A4L-LOC" device=""/>
-<part name="C28" library="rcl" deviceset="C-EU" device="C1206" value="100n"/>
+<part name="C28" library="rcl" deviceset="C-EU" device="C1206" value="10u/35V"/>
 <part name="GND25" library="supply1" deviceset="GND" device=""/>
 <part name="FRAME2" library="frames" deviceset="A4L-LOC" device=""/>
@@
 <part name="FRAME3" library="frames" deviceset="A4L-LOC" device=""/>
 <part name="GND27" library="supply1" deviceset="GND" device=""/>
-<part name="R44" library="resistor" deviceset="R-EU_" device="R0603" value="10k"/>
+<part name="R44" library="resistor" deviceset="R-EU_" device="R0603" value="5k"/>
 <part name="GND29" library="supply1" deviceset="GND" device=""/>
 <part name="SUPPLY7" library="supply2" deviceset="-8V" device=""/>
@@
 <part name="GND20" library="supply1" deviceset="GND" device=""/>
 <part name="+3V13" library="supply1" deviceset="+3V3" device=""/>
-<part name="R12" library="resistor" deviceset="R-EU_" device="R0603" value="10k"/>
+<part name="R12" library="resistor" deviceset="R-EU_" device="R0603" value="n.p."/>
 <part name="R13" library="resistor" deviceset="R-EU_" device="R0603" value="10k"/>
 <part name="R22" library="resistor" deviceset="R-EU_" device="R0603" value="10k"/>
@@
 <part name="+3V14" library="supply1" deviceset="+3V3" device=""/>
 <part name="GND55" library="supply1" deviceset="GND" device=""/>
-<part name="R51" library="resistor" deviceset="R-EU_" device="R0603" value="100k"/>
+<part name="R51" library="resistor" deviceset="R-EU_" device="R0603" value="47k"/>
 <part name="R63" library="resistor" deviceset="R-EU_" device="R0603" value="10k"/>
 <part name="SUPPLY12" library="supply2" deviceset="-8V" device=""/>
